File: WiLoV2/CAD/Eagle/WiLoV2.sch (EAGLE design)
At the start: 139 parts, among them IC1 TPS63060, IC2 MCP73871, J7 U.FL-R-SMT(10), Q1 2N7002, Q2 2N7002, Q3 SI1865DDL-T1-GE3, Q4 NTJD1155LT1G, Q5 NTJD1155LT1G, Q6 NTJD1155LT1G, U1 TPS22917DBVR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

Commit message: Added WiLo V2 dcumentation
Parts:
- S2MINI1: MPN SH2-16G -> (none)
Other:
- note removed: "3.3V Power Supply and Solar Charge Controller"
- note removed: "DHT22 Temperature and Humidity"
- note removed: "DS18B20 Temperature Sensor"
- note removed: "Potentiometer Dendrometer"
- note removed: "Wemos S2 Mini Microcontroller"
